File: ElektronikDevreCizimi(Eagle)/ats.sch (EAGLE design)
At the start: 24 parts, among them IC1 7812TV, IC2 7805TV, Q1 Clock, T1 2N2222, T2 2N2222, U1 ATMEGA328P-PU

Commit message: UpdatedAts
Parts:
- removed C4: 104, ats_lbr:C-US025-025X050
- removed IC1: 7812TV, ats_lbr:7812TV
- removed IC2: 7805TV, ats_lbr:7805TV
- removed R5: 10k, ats_lbr:R-EU_0204/5
- removed SL1: Bzr, con-amp-quick:M02
- removed SL2: Sensor, con-amp-quick:M03
- removed SL3: MainConnect, con-amp-quick:M04
- removed SV3: 3.3VREG, con-lstb:MA03-1
- removed X1: (no value), con-ptr500:AK500/2
- added C9: 0.33 µF, Wurth_Capacitors_WCAP-ATG5-01uf-033uf:WCAP-ATG5_5X11_860020772003
- added J1: 691216510002, 691216510002:691216510002
- added J2: B2B-XH-A(LF)(SN), B2B-XH-A_LF__SN_:B2B-XH-A(LF)(SN)
- added J3: B3B-XH-A_LF__SN_, B3B-XH-A_LF__SN_:B3B-XH-A_LF__SN_
- added J4: B4B-XH-A(LF)(SN), B4B-XH-A_LF__SN_:B4B-XH-A(LF)(SN)
- added R6: 10k, SparkFun-Resistors-10k:10KOHM-HORIZ-1/4W-5%
- added U2: L7812CV, L7812CV:L7812CV
- added U3: L7805CV, L7805CV:L7805CV
- added U4: LM1117T-3.3/NOPB, LM1117T:LM1117T-3.3/NOPB
- C1: value 22 -> 22pF; device ats_lbr:C-US025-025X050 -> SparkFun-Capacitors-01uf:22PF-PTH-2.54MM-200V-5%
- C2: value 22 -> 0.1 µF; device ats_lbr:C-US025-025X050 -> Wurth_Capacitors_WCAP-ATG5-01uf-033uf:WCAP-ATG5_5X11_860020772001
- C3: value 104 -> 22pF; device ats_lbr:C-US025-025X050 -> SparkFun-Capacitors-01uf:22PF-PTH-2.54MM-200V-5%
- C5: value 0.33uf -> 0.1uF; device manken_lbr:C-USBIG050-030X075 -> SparkFun-Capacitors-01uf:0.1UF-KIT-EZ-50V-20%
- C6: value 0.1uf -> 0.1 µF; device manken_lbr:C-USBIG050-030X075 -> Wurth_Capacitors_WCAP-ATG5-01uf-033uf:WCAP-ATG5_5X11_860020772001
- C7: value 10uf -> 0.1uF; device manken_lbr:C-USBIG050-030X075 -> SparkFun-Capacitors-01uf:0.1UF-KIT-EZ-50V-20%
- C8: value 0.1uf -> 10 µF; device manken_lbr:C-USBIG050-030X075 -> Wurth_Capacitors_WCAP-ATG5-01uf-033uf:WCAP-ATG5_5X11_860020372001
- Q1: device ats_lbr:CRYSTALHC49U-V -> adafruitHC-49S(Buyuk):CRYSTALHC49S
- R1, R4: device ats_lbr:R-EU_0204/5 -> SparkFun-Resistors-10k:10KOHM-HORIZ-1/4W-5%
- R2, R3: device ats_lbr:R-EU_0204/5 -> SparkFun-Resistors-1k:1KOHM-HORIZ-1/4W-5%
Connections:
- net 12V: now also C2.+, U2.OUT, U3.INPUT, U4.VIN; no longer C6.1, IC1.VO, IC2.VI, SV3.3
- net 24V: now also C9.+, J1.1, J2.2, U2.IN; no longer C5.1, IC1.VI, SL1.2, X1-1.KL
- net 3.3V: now also C8.+, J3.2, U4.VOUT; no longer C7.1, SL2.2, SV3.2
- net 5V: now also C5.1, C6.+, U3.OUTPUT; no longer C3.1, C8.1, IC2.VO
- net A0: now also J3.3, R6.2; no longer R5.1, SL2.1
- net A4: now also J4.4; no longer SL3.4
- net A5: now also J4.3; no longer SL3.3
- net GND: now also C2.-, C3.1, C6.-, C8.-, C9.-, J1.2, J3.1, J4.1, R6.1, U2.GND, U3.GROUND, U4.GND; no longer C2.1, C3.2, C4.2, C6.2, C8.2, IC1.GND, IC2.GND, R5.2, SL2.3, SL3.1, SV3.1, X1-2.KL
- net N$2: now also J2.1; no longer SL1.1
- net N$4: now also C3.2; no longer C1.2
- net N$5: now also C1.2; no longer C2.2
- net N$6: now also C7.1; no longer C4.1
- net TTKMAIN: now also J4.2; no longer SL3.2
Other:
- moved on the sheet: C1, C3
